File: basketweave/basketweave.kicad_pcb (KiCad board)
At the start: 2 copper layers, 371.5 x 145.3 mm, 177 parts, among them U1 ATmega32A-PU, Y1 16Mhz

Commit message: Working layout 14/05
Parts:
- removed the D71 at (375.5, 119.1)
- removed G***: LOGO, basketweave:logo
- removed REF**: pattern_right, basketweave:pattern_right
- removed REF**: pattern_left, basketweave:pattern_left
- removed RESET: SW_Push, Button_Switch_THT:SW_PUSH_6mm
- removed ROTARY ENCODER: Rotary_Encoder_Switch, Rotary_Encoder:RotaryEncoder_Alps_EC11E-Switch_Vertical_H20mm
- removed USB: GCT-USB-4085-GF-A, Type-C:USB_C_GCT_USB4085
- added D72: D_Small, Diode_THT:D_DO-35_SOD27_P7.62mm_Horizontal, F.Cu at (369.1, 125.6)
- added D73: D_Small, Diode_THT:D_DO-35_SOD27_P7.62mm_Horizontal, F.Cu at (373.9, 143.7)
- added D74: D_Small, Diode_THT:D_DO-35_SOD27_P7.62mm_Horizontal, F.Cu at (378.7, 163.8)
- added D76: D_Small, Diode_THT:D_DO-35_SOD27_P7.62mm_Horizontal, F.Cu at (335.2, 126.6)
- added D78: D_Small, Diode_THT:D_DO-35_SOD27_P7.62mm_Horizontal, F.Cu at (81.4, 185.0)
- added MX72: MX-NoLED, MX_Only:MXOnly-1U-NoLED, F.Cu at (370.7, 115.9)
- added MX73: MX-NoLED, MX_Only:MXOnly-1U-NoLED, F.Cu at (375.4, 134.9)
- added MX74: MX-NoLED, MX_Only:MXOnly-1U-NoLED, F.Cu at (380.2, 154.0)
- added MX75: MX-NoLED, MX_Only:MXOnly-1U-NoLED, F.Cu at (37.3, 154.0)
- added MX76: MX-NoLED, MX_Only:MXOnly-1U-NoLED, F.Cu at (346.9, 118.3)
- added MX77: MX-NoLED, MX_Only:MXOnly-1.25U-NoLED, F.Cu at (58.6, 175.4)
- added MX78: MX-NoLED, MX_Only:MXOnly-1U-NoLED, F.Cu at (80.1, 175.4)
- added MX79: MX-NoLED, MX_Only:MXOnly-ISO-ROTATED-ReversedStabilizers-NoLED, F.Cu at (352.7, 146.9)
- added MX80: MX-NoLED, MX_Only:MXOnly-1U-NoLED, F.Cu at (331.3, 156.4)
- added PATTERN1: Pattern_Left, basketweave:pattern_left, F.Cu at (39.7, 86.5)
- added PATTERN2: Pattern_Right, basketweave:pattern_right, F.Cu at (253.2, 86.5)
- added SW2: RESET, Button_Switch_THT:SW_PUSH_6mm, F.Cu at (221.5, 82.5)
- added SW3: Rotary_Encoder_Switch, basketweave:RotaryEncoder_Alps_EC11E-Switch_Vertical_H20mm-for-MX, F.Cu at (39.8, 146.5)
- added SW4: Rotary_Encoder_Switch, basketweave:RotaryEncoder_Alps_EC11E-Switch_Vertical_H20mm-for-MX, F.Cu at (382.7, 146.5)
- added SW5: Rotary_Encoder_Switch, basketweave:RotaryEncoder_Alps_EC11E-Switch_Vertical_H20mm-for-MX, F.Cu at (49.3, 108.4)
- added SW6: Rotary_Encoder_Switch, basketweave:RotaryEncoder_Alps_EC11E-Switch_Vertical_H20mm-for-MX, F.Cu at (373.2, 108.4)
- added USB1: GCT-USB-4085-GF-A, basketweave:USB_C_GCT_USB4085, F.Cu at (199.2, 82.5)
- F1: footprint cftkb:polyfuse_5.1mm -> basketweave:polyfuse_5.1mm
- SW1: renamed from BOOT; value SW_Push -> BOOT
- moved MX31 292.7 mm to (327.8, 118.3)
- moved D66 3.55 mm to (370.7, 93.7)
- moved D68 3.55 mm to (367.5, 95.3)
- moved MX29 3.48 mm to (326.5, 137.3)
- moved MX28 3.48 mm to (307.5, 137.3)
- moved MX43 1.29 mm to (293.2, 156.4)
- moved MX44 1.29 mm to (312.2, 156.4)
- moved MX27 1.16 mm to (286.1, 136.2)
- moved H2 1.13 mm to (29.4, 101.6)
- moved H4 1.13 mm to (392.9, 101.6)
- moved MX45 1.06 mm to (343.4, 156.6)
- moved MX65 0.96 mm to (271.8, 196.9)
- moved H5 0.83 mm to (164.2, 101.6)
- moved H6 0.83 mm to (234.2, 101.6)
- moved H1 0.76 mm to (29.4, 84.2)
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- renumbered POWER to D71, ISP to J1
Connections:
- D15 pad 2: Net-(D15-Pad2) -> Net-(D15-A)
- D31 pad 2: Net-(D31-Pad2) -> Net-(D31-A)
- D61 pad 2: Net-(D61-Pad2) -> Net-(D61-A)
- D62 pad 2: Net-(D62-Pad2) -> Net-(D62-A)
- MX1 pad 1: COL0 -> unconnected-(MX1-COL-Pad1)
- MX10 pad 1: COL9 -> unconnected-(MX10-COL-Pad1)
- MX11 pad 1: COL10 -> unconnected-(MX11-COL-Pad1)
- MX12 pad 1: COL11 -> unconnected-(MX12-COL-Pad1)
- MX13 pad 1: COL12 -> unconnected-(MX13-COL-Pad1)
- MX14 pad 1: COL13 -> unconnected-(MX14-COL-Pad1)
- MX15 pad 2: Net-(D15-Pad2) -> Net-(D15-A)
- MX16 pad 1: COL0 -> unconnected-(MX16-COL-Pad1)
- MX17 pad 1: COL1 -> unconnected-(MX17-COL-Pad1)
- MX18 pad 1: COL2 -> unconnected-(MX18-COL-Pad1)
- MX19 pad 1: COL3 -> unconnected-(MX19-COL-Pad1)
- MX2 pad 1: COL1 -> unconnected-(MX2-COL-Pad1)
- MX20 pad 1: COL4 -> unconnected-(MX20-COL-Pad1)
- MX21 pad 1: COL5 -> unconnected-(MX21-COL-Pad1)
- MX22 pad 1: COL6 -> unconnected-(MX22-COL-Pad1)
- MX23 pad 1: COL7 -> unconnected-(MX23-COL-Pad1)
- MX24 pad 1: COL8 -> unconnected-(MX24-COL-Pad1)
- MX25 pad 1: COL9 -> unconnected-(MX25-COL-Pad1)
- MX26 pad 1: COL10 -> unconnected-(MX26-COL-Pad1)
- MX27 pad 1: COL11 -> unconnected-(MX27-COL-Pad1)
- MX28 pad 1: COL12 -> unconnected-(MX28-COL-Pad1)
- MX29 pad 1: COL13 -> unconnected-(MX29-COL-Pad1)
- MX3 pad 1: COL2 -> unconnected-(MX3-COL-Pad1)
- MX30 pad 1: COL14 -> unconnected-(MX30-COL-Pad1)
- MX31 pad 1: COL0 -> unconnected-(MX31-COL-Pad1)
- MX31 pad 2: Net-(D31-Pad2) -> Net-(D15-A)
- MX34 pad 1: COL2 -> unconnected-(MX34-COL-Pad1)
- MX35 pad 1: COL3 -> unconnected-(MX35-COL-Pad1)
- MX36 pad 1: COL4 -> unconnected-(MX36-COL-Pad1)
- MX37 pad 1: COL5 -> unconnected-(MX37-COL-Pad1)
- MX38 pad 1: COL6 -> unconnected-(MX38-COL-Pad1)
- MX39 pad 1: COL7 -> unconnected-(MX39-COL-Pad1)
- MX4 pad 1: COL3 -> unconnected-(MX4-COL-Pad1)
- MX40 pad 1: COL8 -> unconnected-(MX40-COL-Pad1)
- MX41 pad 1: COL9 -> unconnected-(MX41-COL-Pad1)
- MX42 pad 1: COL10 -> unconnected-(MX42-COL-Pad1)
- MX43 pad 1: COL11 -> unconnected-(MX43-COL-Pad1)
- MX44 pad 1: COL12 -> unconnected-(MX44-COL-Pad1)
- MX47 pad 1: COL2 -> unconnected-(MX47-COL-Pad1)
- MX49 pad 1: COL4 -> unconnected-(MX49-COL-Pad1)
- MX5 pad 1: COL4 -> unconnected-(MX5-COL-Pad1)
- MX51 pad 1: COL6 -> unconnected-(MX51-COL-Pad1)
- MX53 pad 1: COL8 -> unconnected-(MX53-COL-Pad1)
- MX55 pad 1: COL10 -> unconnected-(MX55-COL-Pad1)
- MX56 pad 1: COL11 -> unconnected-(MX56-COL-Pad1)
- MX57 pad 1: COL12 -> unconnected-(MX57-COL-Pad1)
- MX58 pad 1: COL13 -> unconnected-(MX58-COL-Pad1)
- MX59 pad 1: COL14 -> unconnected-(MX59-COL-Pad1)
- MX6 pad 1: COL5 -> unconnected-(MX6-COL-Pad1)
- MX62 pad 2: Net-(D61-Pad2) -> unconnected-(MX62-ROW-Pad2)
- MX63 pad 2: Net-(D62-Pad2) -> unconnected-(MX63-ROW-Pad2)
- MX7 pad 1: COL6 -> unconnected-(MX7-COL-Pad1)
- MX70 pad 2: Net-(D61-Pad2) -> Net-(D61-A)
- MX71 pad 2: Net-(D62-Pad2) -> Net-(D62-A)
- MX8 pad 1: COL7 -> unconnected-(MX8-COL-Pad1)
- MX9 pad 1: COL8 -> unconnected-(MX9-COL-Pad1)
- U1 pad 14: Net-(U1-Pad14) -> EN_B2
- U1 pad 15: Net-(U1-Pad15) -> EN_B1
- U1 pad 21: EN1 -> unconnected-(U1-PD7-Pad21)
- U1 pad 22: EN2 -> COL15
- U1 pad 32: Net-(U1-Pad32) -> unconnected-(U1-AREF-Pad32)
- U1 pad 4: Net-(U1-Pad4) -> EN_A1
- U1 pad 5: Net-(U1-Pad5) -> EN_A2
Routing:
- net (no net): track 0.00 -> 443.4 mm
- net EN_B1: track 0.00 -> 267.6 mm
- net EN_B2: track 0.00 -> 266.4 mm
- net EN_A1: track 0.00 -> 238.6 mm
- net EN_A2: track 0.00 -> 231.8 mm
- net Net-(D62-Pad2): track 224.7 -> 0.00 mm
- net COL15: track 0.00 -> 209.0 mm
- net Net-(D61-Pad2): track 199.4 -> 0.00 mm
- net EN2: track 166.0 -> 0.00 mm
- net EN1: track 161.3 -> 0.00 mm
- net ROW2: track 436.5 -> 532.7 mm
- net ROW1: track 430.9 -> 517.9 mm, vias 4 -> 3
- net ROW0: track 382.1 -> 462.2 mm
- net Net-(D31-A): track 0.00 -> 79.1 mm
- net GND: track 97.3 -> 26.2 mm, vias 6 -> 10
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Other:
- net class Default removed
- net class Power removed
- board text added: "Based on Basketweave by Noah L github.com/null-ll/basketweave"
- board text added: "Basketweave-S"
- board text added: "JLCJLCJLCJLC"
- board text added: "MX/Encoder1"
- board text added: "MX/Encoder2"
- board text added: "Modified by piit79 of 42keebs.eu github.com/piit79/basketweave-s"
- board text added: "Rev 1.9"
- board text removed: "Designed by Noah L"
- board text removed: "Rev 1"
- board text removed: "github.com/null-ll/basketweave"
