File: basketweave/basketweave.sch (KiCad schematic (older format))
At the start: 174 parts, among them J1 AVR-ISP-6, SW1 SW_Push, SW2 SW_Push, SW3 Rotary_Encoder_Switch, U1 ATmega32A-PU, U2 GCT-USB-4085-GF-A, Y1 16Mhz

Commit message: Working layout 14/05
Parts:
- added D73, D74, D76: D_Small, Diode_THT:D_DO-35_SOD27_P7.62mm_Horizontal, symbol Device:D_Small
- added MX72, MX73, MX74, MX75, MX76: MX-NoLED, MX_Only:MXOnly-1U-NoLED, symbol MX_Alps_Hybrid:MX-NoLED
- added PATTERN1: Pattern_Left, basketweave:pattern_left, symbol Mechanical:MountingHole
- added PATTERN2: Pattern_Right, basketweave:pattern_right, symbol Mechanical:MountingHole
- added SW4, SW5, SW6: Rotary_Encoder_Switch, basketweave:RotaryEncoder_Alps_EC11E-Switch_Vertical_H20mm-for-MX, symbol Device:Rotary_Encoder_Switch
- SW1: value SW_Push -> BOOT
- SW2: value SW_Push -> RESET
- SW3: footprint Rotary_Encoder:RotaryEncoder_Alps_EC11E-Switch_Vertical_H20mm -> basketweave:RotaryEncoder_Alps_EC11E-Switch_Vertical_H20mm-for-MX
- USB1: renamed from U2; symbol Type-C:GCT-USB-4085-GF-A -> Type-C:USB_C_GCT_USB4085-GF-A
Connections:
- net labels added: COL15, EN_A1, EN_A2, EN_B1, EN_B2
- net labels removed: EN1, EN2
- wire segments 230 -> 310
Other:
- note added: "SPLIT BS"
- note removed: "M2"
