File: basketweave_plate/basketweave_plate.kicad_pcb (KiCad board)
At the start: 2 copper layers, 371.5 x 119.1 mm, 1 part

Commit message: Working layout 14/05
Parts:
- G***: footprint basketweave_plate:logo_plate -> basketweave:logo_plate
- moved G*** 1.54 mm to (88.8, 130.1)
Other:
- outline, holes or cut-outs redrawn
- net class Default removed
